File: Hard/control/full/hard_control.sch (KiCad schematic (older format))
At the start: 41 parts, among them IC1 ATMEGA32-P, J1 DB9 FEMALE, P1 CONN_5X2, P2 CONN_5X2, P3 CONN_5X2, P4 CONN_5X2, P5 CONN_5X2, P6 CONN_5X2, U1 MAX202, U2 7805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

Commit message: -Primer propuesta de modificaciones para destello de LEDs de tatami, sin probar. -Archivos kicad adaptados a vesion 2015
Parts:
- C10, C2, C3, C4, C5, C6, C7, C8, C9: symbol C -> C-RESCUE-hard_control
- D1: symbol LED -> LED-RESCUE-hard_control
- R1, R2, R3, R4, R5, R6: symbol R -> R-RESCUE-hard_control
- U1: symbol MAX202 -> MAX202-RESCUE-hard_control
