File: Hard/Kicad_modulo/cartel1.sch (KiCad schematic (older format))
At the start: 42 parts, among them P1 bus, P2 bus, P3 Dinput, P4 Doutput, U1 74LS595, U2 74LS595, U3 74LS595, U4 74LS595

Commit message: Actualización de los esquemáticos a kicad 5.
Parts:
- C1, C2: symbol C -> Device:C
- D1, D10, D11, D12, D13, D14, D15, D16, D17, D18, D19, D2, D20, D21, D22, D23, D24, D25, D26, D27, D28, D29, D3, D30, D31, D32, D4, D5, D6, D7, D8, D9: symbol LED -> Device:LED
- P1, P2: symbol CONN_4X2 -> Connector_Generic:Conn_02x04_Counter_Clockwise
- P3, P4: symbol CONN_1 -> Connector_Generic:Conn_01x01
- U1, U2, U3, U4: symbol 74LS595 -> 74xx:74LS595
Connections:
- wire segments 187 -> 204
Other:
- moved on the sheet: U1, U2, U3, U4
